File: business-card.kicad_pcb (KiCad board)
At the start: 2 copper layers, 85.6 x 54 mm, 14 parts, among them J1 TC2030, U1 NT3H2111W0FHKH

Commit message: Set C1 to 5.1 pF for NFC tuning prototype
The original 1.5pF, I believe, came from an online ST or NXP tool.

The new value comes from FastHenry and FastCap analysis of the actual
PCB coil, feed traces, and nearby copper. Combining the estimated
inductance and parasitic capacitance with the NT3H2111’s nominal 50 pF
input capacitance gives approximately 5.0 pF for NXP’s recommended
14.5 MHz tuning target.

The 5.1 pF used in the schematic predicts a nominal resonance of
approximately 14.48 MHz.
Parts:
- C1: value 1.5pF -> 5.1pF
Changed lines of the file:
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@@
 			)
 		)
-		(property "Value" "1.5pF"
+		(property "Value" "5.1pF"
 			(at 3.3175 0 270)
 			(layer "F.Fab")

Commit message: Update and merges drc for PCBWAY, too
Other:
- rule solder_mask_min_width: 0.13 -> 0.1016
Changed lines of the file:
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@@
 		)
 		(pad_to_mask_clearance 0)
-		(solder_mask_min_width 0.13)
+		(solder_mask_min_width 0.1016)
 		(allow_soldermask_bridges_in_footprints no)
 		(tenting
