File: business-card.kicad_pcb (KiCad board)
At the start: 2 copper layers, 85.6 x 54 mm, 14 parts, among them J1 TC2030, U1 NT3H2111W0FHKH

Commit message: Add additional decoupling cap to tag-connect vcc supply
Not the best placement and routing, but this will be
disabled after debugging.
Parts:
- added C3: 180nF, Capacitor_SMD:C_0402_1005Metric_Pad0.74x0.62mm_HandSolder, F.Cu at (150.1, 95.7)
- C2: value 150nF -> 180nF
Routing:
- net GND: track 57.3 -> 60.7 mm
- net VCC: track 20.5 -> 21.7 mm
