File: business-card.kicad_sch (KiCad schematic)
At the start: 19 parts, among them J1 TC2030, U1 NT3H2111W0FHKH

Commit message: Set C1 to 5.1 pF for NFC tuning prototype
The original 1.5pF, I believe, came from an online ST or NXP tool.

The new value comes from FastHenry and FastCap analysis of the actual
PCB coil, feed traces, and nearby copper. Combining the estimated
inductance and parasitic capacitance with the NT3H2111’s nominal 50 pF
input capacitance gives approximately 5.0 pF for NXP’s recommended
14.5 MHz tuning target.

The 5.1 pF used in the schematic predicts a nominal resonance of
approximately 14.48 MHz.
Parts:
- C1: value 1.5pF -> 5.1pF
Other:
- note added: "C1 originally 1.5 pF. 5.1 pF tuning prototype; verify on assembled PCB."
Changed lines of the file:
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@@
+		)
+	)
+	(text "C1 originally 1.5 pF.\n5.1 pF tuning prototype; verify on assembled PCB."
+		(exclude_from_sim no)
+		(at 77.47 60.96 0)
+		(effects
+			(font
+				(size 1 1)
+			)
+			(justify left)
 		)
 	)
@@
 			)
 		)
-		(property "Value" "1.5pF"
+		(property "Value" "5.1pF"
 			(at 107.95 48.2599 0)
 			(show_name no)

Commit message: Document NFC tuning sensitivity to PCB thickness
Other:
- note added: "C1 originally 1.5 pF. 0.6 mm PCB: 5.1 pF prototype (~14.485 MHz). 0.8 mm PCB: calculated C1 ~4.8 pF for 14.5 MHz; 4.7 pF is the nearest standard E24 value. With 5.1 pF, 0.8 mm resonance is ~14.465 MHz. Assumes nominal 50 pF chip; same copper, FR4 and mask. Verify tuning on assembled PCB with LED load."
- note removed: "C1 originally 1.5 pF. 5.1 pF tuning prototype; verify on assembled PCB."
Changed lines of the file:
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@@
 		)
 	)
-	(text "C1 originally 1.5 pF.\n5.1 pF tuning prototype; verify on assembled PCB."
+	(text "C1 originally 1.5 pF.\n0.6 mm PCB: 5.1 pF prototype (~14.485 MHz).\n0.8 mm PCB: calculated C1 ~4.8 pF for 14.5 MHz;\n4.7 pF is the nearest standard E24 value.\nWith 5.1 pF, 0.8 mm resonance is ~14.465 MHz.\nAssumes nominal 50 pF chip; same copper, FR4 and mask.\nVerify tuning on assembled PCB with LED load."
 		(exclude_from_sim no)
-		(at 77.47 60.96 0)
+		(at 77.47 65.405 0)
 		(effects
 			(font

Commit message: Move contact details to project variables scope
Edit these either in the kicad_pro file OR graphically from the schematic
or PCB setup menu.
Parts:
- INFO1: CONTACT_COMPANY Your Company -> ${PROJ_CONTACT_COMPANY}; CONTACT_EMAIL you@example.com -> ${PROJ_CONTACT_EMAIL}; CONTACT_NAME Your Name -> ${PROJ_CONTACT_NAME}; CONTACT_PHONE +1 202-555-0123 -> ${PROJ_CONTACT_PHONE}; CONTACT_ROLE Your Role -> ${PROJ_CONTACT_ROLE}; CONTACT_WEB example.com -> ${PROJ_CONTACT_WEB}; CONTACT_WEB_QR https://${CONTACT_WEB} -> ${PROJ_CONTACT_WEB_QR}
Changed lines of the file:
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@@
 			)
 		)
-		(property "CONTACT_NAME" "Your Name"
+		(property "CONTACT_NAME" "${PROJ_CONTACT_NAME}"
 			(at 21.59 175.26 0)
 			(show_name no)
@@
 			)
 		)
-		(property "CONTACT_COMPANY" "Your Company"
+		(property "CONTACT_COMPANY" "${PROJ_CONTACT_COMPANY}"
 			(at 21.59 179.07 0)
 			(show_name no)
@@
 			)
 		)
-		(property "CONTACT_ROLE" "Your Role"
+		(property "CONTACT_ROLE" "${PROJ_CONTACT_ROLE}"
 			(at 21.59 182.88 0)
 			(show_name no)
@@
 			)
 		)
-		(property "CONTACT_EMAIL" "you@example.com"
+		(property "CONTACT_EMAIL" "${PROJ_CONTACT_EMAIL}"
 			(at 21.59 187.96 0)
 			(show_name no)
@@
 			)
 		)
-		(property "CONTACT_PHONE" "+1 202-555-0123"
+		(property "CONTACT_PHONE" "${PROJ_CONTACT_PHONE}"
 			(at 21.59 191.77 0)
 			(show_name no)
@@
 			)
 		)
-		(property "CONTACT_WEB" "example.com"
+		(property "CONTACT_WEB" "${PROJ_CONTACT_WEB}"
 			(at 21.59 195.58 0)
 			(show_name no)
@@
 			)
 		)
-		(property "CONTACT_WEB_QR" "https://${CONTACT_WEB}"
+		(property "CONTACT_WEB_QR" "${PROJ_CONTACT_WEB_QR}"
 			(at 44.45 181.61 0)
 			(hide yes)
